File: PCB_files/ext_cons.kicad_sch (KiCad schematic)
At the start: 12 parts, among them J1 Micro_SD_Card_Det1, J2 FFC2B28-40-G, J3 USB_C_Receptacle_USB2.0_14P, J4 CANbus, SW1 nBoot, U4 EMIF06-MSD02N16, U5 TPD8S009DSMR, U6 TPD8S009DSMR, U7 TPD2EUSB30

Commit message: testing updates
D2, D3 part update, PROG direction on boot switch, removed ribbon cable. updated BOM to reflect changes, re-generated gerbers for slight tweaks
Parts:
- SW1: MPN 219G-2ESF -> DS04-254-2-01BK-SMT; Manufacturer CTS -> Same Sky; Reseller_P/N 774-219G-2ESF -> 490-DS04254201BK-SMT
Changed lines of the file:
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@@
 			)
 		)
-		(property "MPN" "219G-2ESF"
+		(property "MPN" "DS04-254-2-01BK-SMT "
 			(at 260.35 99.568 0)
 			(effects
@@
 			)
 		)
-		(property "Reseller_P/N" "774-219G-2ESF"
+		(property "Reseller_P/N" "490-DS04254201BK-SMT"
 			(at 260.35 99.568 0)
 			(effects
@@
 			)
 		)
-		(property "Manufacturer" "CTS"
+		(property "Manufacturer" "Same Sky"
 			(at 260.35 99.568 0)
 			(effects
