File: PCB_files/power.kicad_sch (KiCad schematic)
At the start: 48 parts, among them Q1 DMG2307, Q2 DMG2307, Q3 DMG2307, U3 AP64501SP-13, U9 BD33FC0FP

Commit message: Rev2a initial upload
PCB files
Changed lines of the file:
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@@
 (kicad_sch
-	(version 20231120)
+	(version 20250114)
 	(generator "eeschema")
-	(generator_version "8.0")
+	(generator_version "9.0")
 	(paper "A4")
+	(text "Test Points"
+		(exclude_from_sim no)
+		(at 70.612 101.727 0)
+		(effects
+			(font
+				(size 2.9972 2.9972)
+			)
+			(justify left bottom)
+		)
+	)
+	(text "Place input filter\ncapacitors as close to\nheader as possible"
+		(exclude_from_sim no)
+		(at 27.305 78.867 0)
+		(effects
+			(font
+				(size 1.27 1.27)
+			)
+			(justify left bottom)
+		)
+	)
+	(text "Approx 10mA value for all status LED"
+		(exclude_from_sim no)
+		(at 18.161 149.098 0)
+		(effects
+			(font
+				(size 1.27 1.27)
+			)
+			(justify left bottom)
+		)
+	)
+	(text "Dz protects against\nmax Vgs value"
+		(exclude_from_sim no)
+		(at 54.737 76.708 0)
+		(effects
+			(font
+				(size 1.27 1.27)
+			)
+			(justify left bottom)
+		)
+	)
+	(text "All caps rated at 35V"
+		(exclude_from_sim no)
+		(at 154.94 81.28 0)
+		(effects
+			(font
+				(size 1.27 1.27)
+			)
+			(justify left bottom)
+		)
+	)
+	(text "Design for up to 20V"
+		(exclude_from_sim no)
+		(at 17.272 23.622 0)
+		(effects
+			(font
+				(size 1.27 1.27)
+			)
+			(justify left bottom)
+		)
+	)
+	(text "Input Filter"
+		(exclude_from_sim no)
+		(at 32.004 28.956 0)
+		(effects
+			(font
+				(size 1.27 1.27)
+			)
+			(justify left bottom)
+		)
+	)
+	(text "3v3"
+		(exclude_from_sim no)
+		(at 108.204 102.108 0)
+		(effects
+			(font
+				(size 2.9972 2.9972)
+			)
+			(justify left bottom)
+		)
+	)
+	(text "Dz Voltage spec'd to be slightly lower\nthan max Vin for power IC.\n\nResistors help current limit to prevent\nzener burnout and also lower idle\ncurrent flow for less power disipation."
+		(exclude_from_sim no)
+		(at 81.153 85.344 0)
+		(effects
+			(font
+				(size 1.27 1.27)
+			)
+			(justify left bottom)
+		)
+	)
+	(text "Power Status"
+		(exclude_from_sim no)
+		(at 15.875 101.346 0)
+		(effects
+			(font
+				(size 2.9972 2.9972)
+			)
+			(justify left bottom)
+		)
+	)
+	(text "5v"
+		(exclude_from_sim no)
+		(at 138.176 21.082 0)
+		(effects
+			(font
+				(size 2.9972 2.9972)
+			)
+			(justify left bottom)
+		)
+	)
+	(text "3v3 supply using LDO tested on other boards. \nExpected current draw is max ~200ma.\n\n5V supply taken from CM4 I/O breakout board.\n\nIdeally, a PMOS with higher Vgs than DMG2307 \nwould be better. (Vgs for DMG2307 is rated at \n+/- 30V which could be OK). Doing so would \nprovide more headroom above the Dz Voltage\nprotection vs. Vmax for the FETS"
+		(exclude_from_sim no)
+		(at 112.522 190.246 0)
+		(effects
+			(font
+				(size 1.27 1.27)
+			)
+			(justify left bottom)
+		)
+	)
+	(text "Rev Volt Prot"
+		(exclude_from_sim no)
+		(at 55.245 28.829 0)
+		(effects
+			(font
+				(size 1.27 1.27)
+			)
+			(justify left bottom)
+		)
+	)
+	(text "Over Volt Prot"
+		(exclude_from_sim no)
+		(at 92.329 28.702 0)
+		(effects
+			(font
+				(size 1.27 1.27)
+			)
+			(justify left bottom)
+		)
+	)
+	(text "Power Protection"
+		(exclude_from_sim no)
+		(at 17.018 21.336 0)
+		(effects
+			(font
+				(size 2.9972 2.9972)
+			)
+			(justify left bottom)
+		)
+	)
 	(junction
 		(at 248.285 78.105)
@@
 		)
 	)
-	(text "Test Points"
-		(exclude_from_sim no)
-		(at 70.612 101.727 0)
-		(effects
-			(font
-				(size 2.9972 2.9972)
-			)
-			(justify left bottom)
-		)
-	)
-	(text "Place input filter\ncapacitors as close to\nheader as possible"
-		(exclude_from_sim no)
-		(at 27.305 78.867 0)
-		(effects
-			(font
-				(size 1.27 1.27)
-			)
-			(justify left bottom)
-		)
-	)
-	(text "Approx 10mA value for all status LED"
-		(exclude_from_sim no)
-		(at 18.161 149.098 0)
-		(effects
-			(font
-				(size 1.27 1.27)
-			)
-			(justify left bottom)
-		)
-	)
-	(text "Dz protects against\nmax Vgs value"
-		(exclude_from_sim no)
-		(at 54.737 76.708 0)
-		(effects
-			(font
-				(size 1.27 1.27)
-			)
-			(justify left bottom)
-		)
-	)
-	(text "All caps rated at 35V"
-		(exclude_from_sim no)
-		(at 154.94 81.28 0)
-		(effects
-			(font
-				(size 1.27 1.27)
-			)
-			(justify left bottom)
-		)
-	)
-	(text "Design for up to 20V"
-		(exclude_from_sim no)
-		(at 17.272 23.622 0)
-		(effects
-			(font
-				(size 1.27 1.27)
-			)
-			(justify left bottom)
-		)
-	)
-	(text "Input Filter"
-		(exclude_from_sim no)
-		(at 32.004 28.956 0)
-		(effects
-			(font
-				(size 1.27 1.27)
-			)
-			(justify left bottom)
-		)
-	)
-	(text "3v3"
-		(exclude_from_sim no)
-		(at 108.204 102.108 0)
-		(effects
-			(font
-				(size 2.9972 2.9972)
-			)
-			(justify left bottom)
-		)
-	)
-	(text "Dz Voltage spec'd to be slightly lower\nthan max Vin for power IC.\n\nResistors help current limit to prevent\nzener burnout and also lower idle\ncurrent flow for less power disipation."
-		(exclude_from_sim no)
-		(at 81.153 85.344 0)
-		(effects
-			(font
-				(size 1.27 1.27)
-			)
-			(justify left bottom)
-		)
-	)
-	(text "Power Status"
-		(exclude_from_sim no)
-		(at 15.875 101.346 0)
-		(effects
-			(font
-				(size 2.9972 2.9972)
-			)
-			(justify left bottom)
-		)
-	)
-	(text "5v"
-		(exclude_from_sim no)
-		(at 138.176 21.082 0)
-		(effects
-			(font
-				(size 2.9972 2.9972)
-			)
-			(justify left bottom)
-		)
-	)
-	(text "3v3 supply using LDO tested on other boards. \nExpected current draw is max ~200ma.\n\n5V supply taken from CM4 I/O breakout board.\n\nIdeally, a PMOS with higher Vgs than DMG2307 \nwould be better. (Vgs for DMG2307 is rated at \n+/- 30V which could be OK). Doing so would \nprovide more headroom above the Dz Voltage\nprotection vs. Vmax for the FETS"
-		(exclude_from_sim no)
-		(at 112.522 190.246 0)
-		(effects
-			(font
-				(size 1.27 1.27)
-			)
-			(justify left bottom)
-		)
-	)
-	(text "Rev Volt Prot"
-		(exclude_from_sim no)
-		(at 55.245 28.829 0)
-		(effects
-			(font
-				(size 1.27 1.27)
-			)
-			(justify left bottom)
-		)
-	)
-	(text "Over Volt Prot"
-		(exclude_from_sim no)
-		(at 92.329 28.702 0)
-		(effects
-			(font
-				(size 1.27 1.27)
-			)
-			(justify left bottom)
-		)
-	)
-	(text "Power Protection"
-		(exclude_from_sim no)
-		(at 17.018 21.336 0)
-		(effects
-			(font
-				(size 2.9972 2.9972)
-			)
-			(justify left bottom)
-		)
-	)
 	(label "3v3_in"
 		(at 134.366 118.11 0)
-		(fields_autoplaced yes)
 		(effects
 			(font
@@
 	(label "5v_Vin"
 		(at 178.943 43.18 0)
-		(fields_autoplaced yes)
 		(effects
 			(font
@@
 	(label "Vprot"
 		(at 165.481 43.18 0)
-		(fields_autoplaced yes)
 		(effects
 			(font
@@
 	(label "Vprot"
 		(at 118.618 118.11 0)
-		(fields_autoplaced yes)
 		(effects
 			(font
@@
 	(label "5v_Vin"
 		(at 141.605 73.025 0)
-		(fields_autoplaced yes)
 		(effects
 			(font
@@
 	(label "Vin"
 		(at 33.655 45.72 0)
-		(fields_autoplaced yes)
 		(effects
 			(font
@@
 	(label "Vprot"
 		(at 125.222 45.72 180)
-		(fields_autoplaced yes)
 		(effects
 			(font
@@
 			)
 		)
-		(property "Description" "\nBuck Switching Regulator IC Positive Adjustable 0.8V 1 Output 5A 8-SOIC (0.154, 3.90mm Width) Exposed Pad\n"
+		(property "Description" "Buck Switching Regulator IC Positive Adjustable 0.8V 1 Output 5A 8-SOIC (0.154, 3.90mm Width) Exposed Pad"
 			(at 197.358 49.53 0)
 			(effects
@@
 			)
 		)
-		(property "Datasheet" "293D107X96R3B2TE3 "
+		(property "Datasheet" "293D107X96R3B2TE3"
 			(at 255.27 75.565 0)
 			(effects

Commit message: push from desktop to align files
Parts:
- renumbered C7 to C10, C9 to C11, C14 to C13, C16 to C14, C17 to C15, C18 to C16, C19 to C17, C20 to C18, C4 to C19, C10 to C20, C3 to C21, C8 to C22, C11 to C3, C13 to C4, C1 to C5, C2 to C6, C15 to C7, C5 to C8, C6 to C9, D7 to D2, D4 to D3, D5 to D4, D6 to D5, D1 to D6, D2 to D7, D3 to D8, Q3 to Q2, Q2 to Q3, R2 to R10, R3 to R11, R4 to R12, R9 to R2, R11 to R3, R6 to R4, R10 to R5, R12 to R6, R5 to R8, R8 to R9, TP4 to TP1, TP1 to TP2, TP2 to TP3, TP3 to TP4, U3 to U2, U9 to U3

Commit message: final BOM and tweaking
Tweaked some dimensions after mechanical assembly. Generated BOM and reviewed against reseller inventory
Parts:
- C10, C11, C12, C13, C14, C15, C16, C17, C8, C9: MPN (none) -> C0805C106K4PAC; Manufacturer (none) -> Kemet; Mouser_PN 80-C0805C106K4PAC -> (none); Reseller_P/N (none) -> 80-C0805C106K4PAC; Source/Reseller (none) -> Mouser
- C18: MPN (none) -> TPSB107K010R0400; Manufacturer (none) -> Kyocera; Mouser_PN 581-TPSB107K010R0400 -> (none); Reseller_P/N (none) -> 581-TPSB107K010R0400; Source/Reseller (none) -> Mouser
- C19, C20, C6: MPN (none) -> C0805C105M3RACTU; Manufacturer (none) -> Kemet; Mouser_PN 80-C0805C105M3R -> (none); Reseller_P/N (none) -> 80-C0805C105M3R; Source/Reseller (none) -> Mouser
- C21, C22, C5: MPN (none) -> T495B106K025ATE750; Manufacturer (none) -> Kemet; Mouser_PN 80-T495B106K25ATE750 -> (none); Reseller_P/N (none) -> 80-T495B106K25ATE750; Source/Reseller (none) -> Mouser
- C3, C4: MPN (none) -> C0805C104M5RACTU; Manufacturer (none) -> Kemet; Mouser_PN 80-C0805C104M5R -> (none); Reseller_P/N (none) -> 80-C0805C104M5R; Source/Reseller (none) -> Mouser
- C7: MPN (none) -> C0805C122K5RACTU; Manufacturer (none) -> Kemet; Mouser_PN 80-C0805C122K5R -> (none); Reseller_P/N (none) -> 80-C0805C122K5R; Source/Reseller (none) -> Mouser
- D2, D3, D4, D5: MPN (none) -> MMSZ27T1G; Manufacturer (none) -> OnSemi; Mouser_PN 863-MMSZ27T1G -> (none); Reseller_P/N (none) -> 863-MMSZ27T1G; Source/Reseller (none) -> Mouser
- D6, D7, D8: MPN (none) -> 150080RS75000; Manufacturer (none) -> Wurth; Mouser_PN 710-150080RS75000 -> (none); Reseller_P/N (none) -> 710-150080RS75000; Source/Reseller (none) -> Mouser
- L1: MPN (none) -> SRN6045-3R3Y; Manufacturer (none) -> Bourns; Mouser_PN 652-SRN6045-3R3Y -> (none); Reseller_P/N (none) -> 652-SRN6045-3R3Y; Source/Reseller (none) -> Mouser
- Q1, Q2, Q3: MPN (none) -> DMG2307L-7; Manufacturer (none) -> Diodes; Mouser_PN 621-DMG2307L-7 -> (none); Reseller_P/N (none) -> 621-DMG2307L-7; Source/Reseller (none) -> Mouser
- R10: MPN (none) -> CRCW08052K70FKEA; Manufacturer (none) -> Vishay; Mouser_PN 71-CRCW0805-2.7K-E3 -> (none); Reseller_P/N (none) -> 71-CRCW0805-2.7K-E3; Source/Reseller (none) -> Mouser
- R11: MPN (none) -> CRCW08051K00FKEA; Manufacturer (none) -> Vishay; Mouser_PN 71-CRCW0805-1.0K-E3 -> (none); Reseller_P/N (none) -> 71-CRCW0805-1.0K-E3; Source/Reseller (none) -> Mouser
- R12: MPN (none) -> CRCW0805665RFKEA; Manufacturer (none) -> Vishay; Mouser_PN 71-CRCW0805-665-E3 -> (none); Reseller_P/N (none) -> 71-CRCW0805-665-E3; Source/Reseller (none) -> Mouser
- R2: MPN (none) -> CRCW080510R0FKEA; Manufacturer (none) -> Vishay; Mouser_PN 71-CRCW0805-10-E3 -> (none); Reseller_P/N (none) -> 71-CRCW0805-10-E3; Source/Reseller (none) -> Mouser
- R3: MPN (none) -> CRCW080512K0FKTA; Manufacturer (none) -> Vishay; Mouser_PN 71-CRCW0805-12K -> (none); Reseller_P/N (none) -> 71-CRCW0805-12K; Source/Reseller (none) -> Mouser
- R4, R7, R8, R9: MPN (none) -> CRCW080510K0FKEA; Manufacturer (none) -> Vishay; Mouser_PN 71-CRCW0805-10K-E3 -> (none); Reseller_P/N (none) -> 71-CRCW0805-10K-E3; Source/Reseller (none) -> Mouser
- R5: MPN (none) -> CRCW080520K0FKEA; Manufacturer (none) -> Vishay; Mouser_PN 71-CRCW0805-20K-E3 -> (none); Reseller_P/N (none) -> 71-CRCW0805-20K-E3; Source/Reseller (none) -> Mouser
- R6: MPN (none) -> CRCW08052K20FKEA; Manufacturer (none) -> Vishay; Mouser_PN 71-CRCW0805-2.2K-E3 -> (none); Reseller_P/N (none) -> 71-CRCW0805-2.2K-E3; Source/Reseller (none) -> Mouser
- TP1, TP2, TP3, TP4: Mouser_PN N/A -> (none); Reseller_P/N (none) -> N/A; Source/Reseller (none) -> N/A; now left out of the parts list
- U2: MPN (none) -> AP64501SP-13; Manufacturer Diodes Incorporated -> Diodes; Mouser_PN 621-AP64501SP-13 -> (none); Reseller_P/N (none) -> 621-AP64501SP-13; Source/Reseller (none) -> Mouser
- U3: MPN (none) -> NCV1117DT33T5G; Manufacturer (none) -> OnSemi; Mouser_PN 755-BD33FC0FP-E2 -> (none); Reseller_P/N (none) -> 863-NCV1117DT33T5G; Source/Reseller (none) -> Mouser
