File: PCB_files/power.kicad_sch (KiCad schematic)
At the start: 48 parts, among them Q1 DMG2307, Q2 DMG2307, Q3 DMG2307, U2 AP64501SP-13, U3 BD33FC0FP

Commit message: testing updates
D2, D3 part update, PROG direction on boot switch, removed ribbon cable. updated BOM to reflect changes, re-generated gerbers for slight tweaks
Parts:
- D2, D3: value 27V -> 2A 60V; MPN MMSZ27T1G -> CDBMT260-HF; Manufacturer OnSemi -> Comchip; Reseller_P/N 863-MMSZ27T1G -> 750-CDBMT260-HF
Changed lines of the file:
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@@
 			)
 		)
-		(property "Value" "27V"
+		(property "Value" "2A 60V"
 			(at 175.768 40.2336 0)
 			(effects
@@
 			)
 		)
-		(property "MPN" "MMSZ27T1G"
+		(property "MPN" "CDBMT260-HF"
 			(at 175.768 43.18 0)
 			(effects
@@
 			)
 		)
-		(property "Reseller_P/N" "863-MMSZ27T1G"
+		(property "Reseller_P/N" "750-CDBMT260-HF"
 			(at 175.768 43.18 0)
 			(effects
@@
 			)
 		)
-		(property "Manufacturer" "OnSemi"
+		(property "Manufacturer" "Comchip"
 			(at 175.768 43.18 0)
 			(effects
@@
 			)
 		)
-		(property "Value" "27V"
+		(property "Value" "2A 60V"
 			(at 68.199 51.0286 0)
 			(effects
@@
 			)
 		)
-		(property "MPN" "MMSZ27T1G"
+		(property "MPN" "CDBMT260-HF"
 			(at 68.199 53.975 0)
 			(effects
@@
 			)
 		)
-		(property "Reseller_P/N" "863-MMSZ27T1G"
+		(property "Reseller_P/N" "750-CDBMT260-HF"
 			(at 68.199 53.975 0)
 			(effects
@@
 			)
 		)
-		(property "Manufacturer" "OnSemi"
+		(property "Manufacturer" "Comchip"
 			(at 68.199 53.975 0)
 			(effects
