File: PCB_files/mechanical.kicad_sch (KiCad schematic)
At the start: 34 parts, among them J10 12x12 keycap - white, J11 12x12 keycap - white, J12 12x12 keycap - white, J13 12x12 keycap - white, J14 12x12 keycap - white, J5 CM4-A, J6 CM4-B, J7 HDMI_ribbon, J8 HDMI_Display, J9 12x12 keycap - white

Commit message: testing updates
D2, D3 part update, PROG direction on boot switch, removed ribbon cable. updated BOM to reflect changes, re-generated gerbers for slight tweaks
Parts:
- removed J7: HDMI_ribbon, N/A, symbol Connector_Generic:Conn_01x01
Changed lines of the file:
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@@
-	)
-	(symbol
-		(lib_id "Connector_Generic:Conn_01x01")
-		(at 108.458 88.138 0)
-		(unit 1)
-		(exclude_from_sim no)
-		(in_bom yes)
-		(on_board no)
-		(dnp no)
-		(fields_autoplaced yes)
-		(property "Reference" "J7"
-			(at 111.506 86.8679 0)
-			(effects
-				(font
-					(size 1.27 1.27)
-				)
-				(justify left)
-			)
-		)
-		(property "Value" "HDMI_ribbon"
-			(at 111.506 89.4079 0)
-			(effects
-				(font
-					(size 1.27 1.27)
-				)
-				(justify left)
-			)
-		)
-		(property "Footprint" "N/A"
-			(at 108.458 88.138 0)
-			(effects
-				(font
-					(size 1.27 1.27)
-				)
-				(hide yes)
-			)
-		)
-		(property "Datasheet" "~"
-			(at 108.458 88.138 0)
-			(effects
-				(font
-					(size 1.27 1.27)
-				)
-				(hide yes)
-			)
-		)
-		(property "Description" "40 pin 0.5mm pitch FFC"
-			(at 108.458 88.138 0)
-			(effects
-				(font
-					(size 1.27 1.27)
-				)
-				(hide yes)
-			)
-		)
-		(property "MPN" "05-40-D-0152-A-4-06-4-G"
-			(at 108.458 88.138 0)
-			(effects
-				(font
-					(size 1.27 1.27)
-				)
-				(hide yes)
-			)
-		)
-		(property "OC_FARNELL" ""
-			(at 108.458 88.138 0)
-			(effects
-				(font
-					(size 1.27 1.27)
-				)
-				(hide yes)
-			)
-		)
-		(property "OC_NEWARK" ""
-			(at 108.458 88.138 0)
-			(effects
-				(font
-					(size 1.27 1.27)
-				)
-				(hide yes)
-			)
-		)
-		(property "PACKAGE" ""
-			(at 108.458 88.138 0)
-			(effects
-				(font
-					(size 1.27 1.27)
-				)
-				(hide yes)
-			)
-		)
-		(property "SUPPLIER" ""
-			(at 108.458 88.138 0)
-			(effects
-				(font
-					(size 1.27 1.27)
-				)
-				(hide yes)
-			)
-		)
-		(property "Sim.Device" ""
-			(at 108.458 88.138 0)
-			(effects
-				(font
-					(size 1.27 1.27)
-				)
-				(hide yes)
-			)
-		)
-		(property "Sim.Pins" ""
-			(at 108.458 88.138 0)
-			(effects
-				(font
-					(size 1.27 1.27)
-				)
-				(hide yes)
-			)
-		)
-		(property "Reseller_P/N" "640-540-D0152A4064T"
-			(at 108.458 88.138 0)
-			(effects
-				(font
-					(size 1.27 1.27)
-				)
-				(hide yes)
-			)
-		)
-		(property "Source/Reseller" "Mouser"
-			(at 108.458 88.138 0)
-			(effects
-				(font
-					(size 1.27 1.27)
-				)
-				(hide yes)
-			)
-		)
-		(property "Manufacturer" "GCT"
-			(at 108.458 88.138 0)
-			(effects
-				(font
-					(size 1.27 1.27)
-				)
-				(hide yes)
-			)
-		)
-		(pin "1"
-		)
-		(instances
-			(project "py_dash_pcb_7"
-				(path "/84878699-1e21-48de-ad1b-9d4034e33e81/bd67a017-df07-4337-876d-8f0fee0733f5"
-					(reference "J7")
-					(unit 1)
-				)
-			)
-		)
 	)
 	(symbol
