File: PCB_files/perif.kicad_sch (KiCad schematic)
At the start: 35 parts, among them SW2 SW_Push, SW3 SW_Push, SW4 SW_Push, SW5 SW_Push, SW6 SW_Push, SW7 SW_Push, U8 MCP2515-xST, U9 SN65HVD234, Y1 16Mhz

Commit message: BOM update
part number corrections
Parts:
- U9: value SN65HVD234 -> SN65HVD231; MPN SN65HVD234DR -> SN65HVD231D; Reseller_P/N 595-SN65HVD234DR -> 595-SN65HVD231D
Other:
- note added: "U9 can be replaced with a SN65HCD234 chip, however pin 5 must be tied to vcc."
Changed lines of the file:
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@@
+		)
+	)
+	(text "U9 can be replaced with a SN65HCD234\nchip, however pin 5 must be tied to vcc."
+		(exclude_from_sim no)
+		(at 26.162 125.476 0)
+		(effects
+			(font
+				(size 1.27 1.27)
+			)
+			(justify left bottom)
 		)
 	)
@@
 			)
 		)
-		(property "Value" "SN65HVD234"
+		(property "Value" "SN65HVD231"
 			(at 41.91 93.345 0)
 			(effects
@@
 			)
 		)
-		(property "Datasheet" "http://www.ti.com/lit/ds/symlink/sn65hvd234.pdf"
+		(property "Datasheet" "http://www.ti.com/lit/ds/symlink/sn65hvd231.pdf"
 			(at 54.61 90.17 0)
 			(effects
@@
 			)
 		)
-		(property "MPN" "SN65HVD234DR"
+		(property "MPN" "SN65HVD231D"
 			(at 57.15 100.33 0)
 			(effects
@@
 			)
 		)
-		(property "Reseller_P/N" "595-SN65HVD234DR"
+		(property "Reseller_P/N" "595-SN65HVD231D"
 			(at 57.15 100.33 0)
 			(effects
